File: PCB/PCB_Back/WS2812B.kicad_sch (KiCad schematic)
At the start: 30 parts

Commit message: Layout, Routing, Stuff
Connections:
- net at D3.2 (DOUT): now also D4.4 (DIN); no longer D6.4 (DIN)
- net at D3.4 (DIN): now also D2.2 (DOUT); no longer D14.2 (DOUT)
- net at D9.2 (DOUT): now also D10.4 (DIN); no longer D12.4 (DIN)
- net at D9.4 (DIN): now also D8.2 (DOUT); no longer D6.2 (DOUT)
- net at D7.4 (DIN): now also D6.2 (DOUT); no longer D4.2 (DOUT)
- net at D1.2 (DOUT): now also D2.4 (DIN); no longer D4.4 (DIN)
- net at D10.2 (DOUT): now also D11.4 (DIN); no longer D13.4 (DIN)
- net at D7.2 (DOUT): now also D8.4 (DIN); no longer D10.4 (DIN)
- net at D11.2 (DOUT): now also D12.4 (DIN); no longer D14.4 (DIN)
- net at D15.4 (DIN): now also D14.2 (DOUT); no longer D12.2 (DOUT)
- net at D5.4 (DIN): now also D4.2 (DOUT); no longer D2.2 (DOUT)
- net at D13.2 (DOUT): now also D14.4 (DIN); no longer D2.4 (DIN)
- net at D5.2 (DOUT): now also D6.4 (DIN); no longer D8.4 (DIN)
- new net: D12.2 (DOUT), D13.4 (DIN)
Other:
- moved on the sheet: D10, D11, D12, D13, D14, D2, D3, D4, D5, D6, D7, D9
